File: eesc/CAN.kicad_sch (KiCad schematic)
At the start: 0 parts

Commit message: Most updated changes
Parts:
- added C52, C53: 2.2u, symbol Device:C
- added J6: CAN, symbol Connector_Generic:Conn_01x04
- added R33: 220, symbol Device:R
- added U8: TJA1051TK-3, Package_DFN_QFN:DFN-8-1EP_3x3mm_P0.65mm_EP1.55x2.4mm, symbol Interface_CAN_LIN:TJA1051TK-3
Connections:
- new net: C52.2, C53.2, J6.1 (Pin_1), U8.2 (GND), U8.8 (S), U8.9 (GND)
- new net +3.3V: C53.1, U8.5 (VIO)
- new net +5V: C52.1, J6.4 (Pin_4), U8.3 (VCC)
- new net CAN+: J6.3 (Pin_3), R33.1, U8.7 (CANH)
- new net CAN-: J6.2 (Pin_2), R33.2, U8.6 (CANL)
- new net RX: U8.4 (RXD)
- new net TX: U8.1 (TXD)
