File: eesc/DRV8301.kicad_sch (KiCad schematic)
At the start: 0 parts

Commit message: Add current sense and finish DRV8301 Circuit
Parts:
- added C33: 15n, Capacitor_SMD:C_0603_1608Metric, symbol Device:C
- added C33: 120p, Capacitor_SMD:C_0603_1608Metric, symbol Device:C
- added C33 (x3), C45 (x4): 2.2u, Capacitor_SMD:C_0603_1608Metric, symbol Device:C
- added C33: 6.8n, Capacitor_SMD:C_0603_1608Metric, symbol Device:C
- added C33, C45: 4.7u100v, Capacitor_SMD:C_0603_1608Metric, symbol Device:C
- added C34: 100n, Capacitor_SMD:C_0603_1608Metric, symbol Device:C
- added C35: 4.7u, Capacitor_THT:CP_Radial_D4.0mm_P1.50mm, symbol Device:C_Polarized
- added C35: 100u, Capacitor_THT:CP_Radial_D4.0mm_P1.50mm, symbol Device:C_Polarized
- added C36, C38, C40: 220n, Capacitor_SMD:C_0603_1608Metric, symbol Device:C
- added C39: 22n, Capacitor_SMD:C_0603_1608Metric, symbol Device:C
- added D1: 1N5819, Diode_SMD:D_SMA, symbol Diode:1N5819
- added D2: TVS, symbol Device:D
- added L1: 22u, Inductor_SMD:L_Taiyo-Yuden_NR-30xx, symbol pspice:INDUCTOR
- added R1: 220k, symbol Device:R
- added R14, R5: 10k, symbol Device:R
- added R2: 15k, symbol Device:R
- added R3: 18k, symbol Device:R
- added R4: 3.3k, symbol Device:R
- added U2: DRV8301DCAR, Package_SO:HTSSOP-56-1EP_6.1x14mm_P0.5mm_EP3.61x6.35mm, symbol DRV8301DCAR:DRV8301DCAR
- added U3: AMS1117-3.3, Package_TO_SOT_SMD:SOT-223-3_TabPin2, symbol Regulator_Linear:AMS1117-3.3
Connections:
- new net: C33.2, U2.56 (SS_TR)
- new net: C34.2, D1.1 (K), L1.1, U2.50 (PH_1), U2.51 (PH_2)
- new net: C33.2, R2.2, U2.2 (COMP)
- new net: C39.1, U2.15 (CP2)
- new net: C39.2, U2.14 (CP1)
- new net: C40.1, U2.38 (BST_C)
- new net: C36.1, U2.48 (BST_A)
- new net: C45.1, C45.1, U2.13 (GVDD)
- new net: C45.1, U2.23 (DVDD)
- new net: R5.2, U2.7 (DTC)
- new net: C34.1, U2.52 (BST_BK)
- new net: C33.2, R2.1
- new net: R3.2, R4.1, U2.3 (VSENSE)
- new net: R1.2, U2.1 (RT_CLK)
- new net: C45.1, U2.24 (REF), U2.27 (AVDD)
- new net: C38.1, U2.43 (BST_B)
- new net +3.3V: C33.1, C35.1, U2.49 (VDD_SPI), U3.2 (VO)
- new net +5V: C33.1, C33.1, C35.1, D2.1 (K), L1.2, R3.1, U3.3 (VI)
- new net CS: U2.8 (N_SCS)
- new net EN_BUCK: U2.55 (EN_BUCK)
- new net EN_GATE: R14.2, U2.16 (EN_GATE)
- new net FAULT: U2.6 (N_FAULT)
- new net GH_A: U2.47 (GH_A)
- new net GH_B: U2.42 (GH_B)
- new net GH_C: U2.37 (GH_C)
- new net GL_A: U2.45 (GL_A)
- new net GL_B: U2.40 (GL_B)
- new net GL_C: U2.35 (GL_C)
- new net GND: C33.1, C33.1, C33.1, C33.1, C33.2, C33.2, C33.2, C35.2, C35.2, C45.2, C45.2, C45.2, C45.2, C45.2, D1.2 (A), D2.2 (A), R1.1, R14.1, R4.2, R5.1, U2.28 (AGND), U2.30 (SP2), U2.31 (SN2), U2.32 (SP1), U2.33 (SN1), U2.57 (EP), U3.1 (GND)
- new net INH_A: U2.17 (INH_A)
- new net INH_B: U2.19 (INH_B)
- new net INH_C: U2.21 (INH_C)
- new net INL_B: U2.18 (INL_A), U2.20 (INL_B)
- new net INL_C: U2.22 (INL_C)
- new net SCLK: U2.11 (SCLK)
- new net SD0: U2.10 (SDO)
- new net SDI: U2.9 (SDI)
- new net SH_A: C36.2, U2.46 (SH_A)
- new net SH_B: C38.2, U2.41 (SH_B)
- new net SH_C: C40.2, U2.36 (SH_C)
- new net SL_A: U2.44 (SL_A)
- new net SL_B: U2.39 (SL_B)
- new net SL_C: U2.34 (SL_C)
- new net V_SUPPLY: C33.2, C45.1, U2.29 (PVDD1), U2.53 (PVDD2_1), U2.54 (PVDD2_2)
- no-connect marks 0 -> 5
Other:
- note added: "5V to 3.3V Linear Regulator"
- note added: "Transient Protection"

Commit message: Complete transistor stage
Parts:
- removed C33: 2.2u, Capacitor_SMD:C_0603_1608Metric, symbol Device:C
- removed D1: 1N5819, Diode_SMD:D_SMA, symbol Diode:1N5819
- added D3: B160, Diode_SMD_AKL:D_SMA, symbol PCM_Diode_Schottky_AKL:B160
Connections:
- net GND: now also D3.2 (A)
- net at C34.2, L1.1, U2.50 (PH_1)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: now also D3.1 (K)
Other:
- moved on the sheet: C33, C34, C35, C36, C38, C39, C40, C45, D2, L1, R1, R14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

Commit message: Most updated changes
Parts:
- added C33: 2.2u, Capacitor_SMD:C_0603_1608Metric, symbol Device:C
Connections:
- net +5V: now also C33.1
- net GND: now also C33.2
Other:
- moved on the sheet: R3, R4
Changed lines of the file:
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@@
   (junction (at 116.205 129.54) (diameter 0) (color 0 0 0 0)
   )
+  (junction (at 212.09 86.36) (diameter 0) (color 0 0 0 0)
+  )
   (junction (at 96.52 78.74) (diameter 0) (color 0 0 0 0)
   )
@@
   (junction (at 79.375 105.41) (diameter 0) (color 0 0 0 0)
   )
-  (junction (at 211.455 86.36) (diameter 0) (color 0 0 0 0)
-  )
   (junction (at 174.625 68.58) (diameter 0) (color 0 0 0 0)
   )
@@
   (junction (at 163.195 124.46) (diameter 0) (color 0 0 0 0)
   )
-  (junction (at 211.455 73.66) (diameter 0) (color 0 0 0 0)
+  (junction (at 212.09 73.66) (diameter 0) (color 0 0 0 0)
   )
   (junction (at 165.735 132.08) (diameter 0) (color 0 0 0 0)
@@
     (stroke (width 0) (type default))
   )
-  (wire (pts (xy 207.645 73.66) (xy 211.455 73.66))
+  (wire (pts (xy 207.645 73.66) (xy 212.09 73.66))
     (stroke (width 0) (type default))
   )
@@
     (stroke (width 0) (type default))
   )
+  (wire (pts (xy 212.09 86.36) (xy 222.885 86.36))
+    (stroke (width 0) (type default))
+  )
   (wire (pts (xy 125.095 121.92) (xy 116.205 121.92))
     (stroke (width 0) (type default))
@@
     (stroke (width 0) (type default))
   )
+  (wire (pts (xy 212.09 73.66) (xy 212.09 76.2))
+    (stroke (width 0) (type default))
+  )
   (wire (pts (xy 179.705 73.66) (xy 179.705 78.74))
     (stroke (width 0) (type default))
@@
     (stroke (width 0) (type default))
   )
+  (wire (pts (xy 212.09 73.66) (xy 222.885 73.66))
+    (stroke (width 0) (type default))
+  )
   (wire (pts (xy 174.625 109.22) (xy 177.165 109.22))
     (stroke (width 0) (type default))
@@
     (stroke (width 0) (type default))
   )
-  (wire (pts (xy 211.455 86.36) (xy 222.885 86.36))
-    (stroke (width 0) (type default))
-  )
   (wire (pts (xy 105.41 144.78) (xy 116.205 144.78))
     (stroke (width 0) (type default))
@@
     (stroke (width 0) (type default))
   )
-  (wire (pts (xy 211.455 73.66) (xy 222.885 73.66))
-    (stroke (width 0) (type default))
-  )
   (wire (pts (xy 224.155 111.125) (xy 232.41 111.125))
     (stroke (width 0) (type default))
@@
     (stroke (width 0) (type default))
   )
+  (wire (pts (xy 96.52 66.04) (xy 96.52 68.58))
+    (stroke (width 0) (type default))
+  )
   (wire (pts (xy 160.655 101.6) (xy 177.165 101.6))
     (stroke (width 0) (type default))
@@
     (stroke (width 0) (type default))
   )
-  (wire (pts (xy 96.52 68.58) (xy 96.52 67.945))
-    (stroke (width 0) (type default))
-  )
   (wire (pts (xy 191.135 73.66) (xy 191.135 76.2))
     (stroke (width 0) (type default))
@@
     (stroke (width 0) (type default))
   )
-  (wire (pts (xy 191.135 86.36) (xy 211.455 86.36))
+  (wire (pts (xy 191.135 86.36) (xy 212.09 86.36))
     (stroke (width 0) (type default))
   )
@@
     (stroke (width 0) (type default))
   )
-  (wire (pts (xy 211.455 84.455) (xy 211.455 86.36))
-    (stroke (width 0) (type default))
-  )
   (wire (pts (xy 121.285 58.42) (xy 121.285 63.5))
     (stroke (width 0) (type default))
@@
     (stroke (width 0) (type default))
   )
+  (wire (pts (xy 212.09 83.82) (xy 212.09 86.36))
+    (stroke (width 0) (type default))
+  )
   (wire (pts (xy 114.3 45.72) (xy 121.285 45.72))
     (stroke (width 0) (type default))
@@
     (stroke (width 0) (type default))
   )
+  (wire (pts (xy 96.52 69.85) (xy 96.52 68.58))
+    (stroke (width 0) (type default))
+  )
   (wire (pts (xy 125.095 93.98) (xy 90.17 93.98))
     (stroke (width 0) (type default))
@@
     (stroke (width 0) (type default))
   )
-  (wire (pts (xy 96.52 57.15) (xy 96.52 60.325))
+  (wire (pts (xy 96.52 57.15) (xy 96.52 58.42))
     (stroke (width 0) (type default))
   )
@@
     (stroke (width 0) (type default))
   )
-  (wire (pts (xy 96.52 78.74) (xy 96.52 76.2))
+  (wire (pts (xy 96.52 78.74) (xy 96.52 77.47))
     (stroke (width 0) (type default))
   )
@@
   )
   (wire (pts (xy 160.655 76.2) (xy 161.925 76.2))
-    (stroke (width 0) (type default))
-  )
-  (wire (pts (xy 211.455 73.66) (xy 211.455 76.835))
     (stroke (width 0) (type default))
   )
@@
     )
   )
+  (symbol (lib_id "Device:C") (at 212.09 80.01 0) (unit 1)
+    (in_bom yes) (on_board yes) (dnp no) (fields_autoplaced)
+    (property "Reference" "C33" (at 215.265 79.375 0)
+      (effects (font (size 1.27 1.27)) (justify left))
+    )
+    (property "Value" "2.2u" (at 215.265 81.915 0)
+      (effects (font (size 1.27 1.27)) (justify left))
+    )
+    (property "Footprint" "Capacitor_SMD:C_0603_1608Metric" (at 213.0552 83.82 0)
+      (effects (font (size 1.27 1.27)) hide)
+    )
+    (property "Datasheet" "~" (at 212.09 80.01 0)
+      (effects (font (size 1.27 1.27)) hide)
+    )
+    (pin "1")
+    (pin "2")
+    (instances
+      (project "electrium-esc"
+        (path "/d277d506-2f4d-497b-a498-1ff059e212d2/4dcd2554-0c0c-4fca-b220-d2fb156d9cf9"
+          (reference "C33") (unit 1)
+        )
+        (path "/d277d506-2f4d-497b-a498-1ff059e212d2/8c1d7bfe-a7ad-4b08-9e6d-dd7b239bc0ed"
+          (reference "C56") (unit 1)
+        )
+      )
+      (project "eesc"
+        (path "/ef2a3433-a5aa-4be9-bc22-47192e2652e7/40141f3c-7306-421f-947e-a976cd111365"
+          (reference "C48") (unit 1)
+        )
+      )
+    )
+  )
   (symbol (lib_id "Device:C_Polarized") (at 267.335 116.84 0) (unit 1)
     (in_bom yes) (on_board yes) (dnp no) (fields_autoplaced)
@@
     )
   )
-  (symbol (lib_id "Device:R") (at 96.52 72.39 0) (unit 1)
-    (in_bom yes) (on_board yes) (dnp no) (fields_autoplaced)
-    (property "Reference" "R4" (at 98.425 71.755 0)
-      (effects (font (size 1.27 1.27)) (justify left))
-    )
-    (property "Value" "3.3k" (at 98.425 74.295 0)
-      (effects (font (size 1.27 1.27)) (justify left))
-    )
-    (property "Footprint" "" (at 94.742 72.39 90)
-      (effects (font (size 1.27 1.27)) hide)
-    )
-    (property "Datasheet" "~" (at 96.52 72.39 0)
+  (symbol (lib_id "Device:R") (at 96.52 73.66 0) (unit 1)
+    (in_bom yes) (on_board yes) (dnp no) (fields_autoplaced)
+    (property "Reference" "R4" (at 98.425 73.025 0)
+      (effects (font (size 1.27 1.27)) (justify left))
+    )
+    (property "Value" "3.3k" (at 98.425 75.565 0)
+      (effects (font (size 1.27 1.27)) (justify left))
+    )
+    (property "Footprint" "" (at 94.742 73.66 90)
+      (effects (font (size 1.27 1.27)) hide)
+    )
+    (property "Datasheet" "~" (at 96.52 73.66 0)
       (effects (font (size 1.27 1.27)) hide)
     )
@@
     )
   )
-  (symbol (lib_id "Device:R") (at 96.52 64.135 0) (unit 1)
-    (in_bom yes) (on_board yes) (dnp no) (fields_autoplaced)
-    (property "Reference" "R3" (at 98.425 63.5 0)
-      (effects (font (size 1.27 1.27)) (justify left))
-    )
-    (property "Value" "18k" (at 98.425 66.04 0)
-      (effects (font (size 1.27 1.27)) (justify left))
-    )
-    (property "Footprint" "" (at 94.742 64.135 90)
-      (effects (font (size 1.27 1.27)) hide)
-    )
-    (property "Datasheet" "~" (at 96.52 64.135 0)
-      (effects (font (size 1.27 1.27)) hide)
-    )
+  (symbol (lib_id "Device:R") (at 96.52 62.23 0) (unit 1)
+    (in_bom yes) (on_board yes) (dnp no) (fields_autoplaced)
+    (property "Reference" "R3" (at 98.425 61.595 0)
+      (effects (font (size 1.27 1.27)) (justify left))
+    )
+    (property "Value" "18k" (at 98.425 64.135 0)
+      (effects (font (size 1.27 1.27)) (justify left))
+    )
+    (property "Footprint" "" (at 94.742 62.23 90)
+      (effects (font (size 1.27 1.27)) hide)
+    )
+    (property "Datasheet" "~" (at 96.52 62.23 0)
+      (effects (font (size 1.27 1.27)) hide)
+    )
