File: eesc/Hall.kicad_sch (KiCad schematic)
At the start: 0 parts

Commit message: Most updated changes
Parts:
- added C49: 100n, symbol Device:C
- added J5: Hall, symbol Connector_Generic:Conn_01x06
- added R27, R28, R29: 2.2k, symbol Device:R
- added R30: 10k, symbol Device:R
- added SW1: HALL_VOLT, symbol Switch:SW_DPDT_x2
Connections:
- new net: J5.6 (Pin_6), R27.1, R28.1, R29.1, SW1.2 (B)
- new net +3.3V: R30.1, SW1.1 (A)
- new net +5V: SW1.3 (C)
- new net GND: C49.1, J5.1 (Pin_1)
- new net HALL_1: J5.4 (Pin_4), R29.2
- new net HALL_2: J5.3 (Pin_3), R28.2
- new net HALL_3: J5.2 (Pin_2), R27.2
- new net HALL_TEMP: C49.2, J5.5 (Pin_5), R30.2
