File: eesc/IMU.kicad_sch (KiCad schematic)
At the start: 0 parts

Commit message: Most updated changes
Parts:
- added C50, C51: 2.2u, symbol Device:C
- added U7: BMI160, Package_LGA:Bosch_LGA-14_3x2.5mm_P0.5mm, symbol Sensor_Motion:BMI160
Connections:
- new net +3.3V: C50.1, C51.1, U7.12 (CSB), U7.5 (VDDIO), U7.8 (VDD)
- new net GND: C50.2, C51.2, U7.1 (SDO), U7.6 (GNDIO), U7.7 (GND)
- new net SCL: U7.13 (SCx)
- new net SDA: U7.14 (SDx)
- no-connect marks 0 -> 4
Changed lines of the file:
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@@
 (kicad_sch (version 20230121) (generator eeschema)
   (paper "A4")
+  (junction (at 142.24 114.3) (diameter 0) (color 0 0 0 0)
+  )
+  (junction (at 160.02 114.3) (diameter 0) (color 0 0 0 0)
+  )
+  (junction (at 142.24 83.82) (diameter 0) (color 0 0 0 0)
+  )
+  (junction (at 144.78 114.3) (diameter 0) (color 0 0 0 0)
+  )
+  (junction (at 144.78 83.82) (diameter 0) (color 0 0 0 0)
+  )
+  (junction (at 160.02 83.82) (diameter 0) (color 0 0 0 0)
+  )
+  (no_connect (at 154.94 100.33))
+  (no_connect (at 154.94 97.79))
+  (no_connect (at 154.94 102.87))
+  (no_connect (at 154.94 95.25))
+  (wire (pts (xy 144.78 83.82) (xy 160.02 83.82))
+    (stroke (width 0) (type default))
+  )
+  (wire (pts (xy 142.24 114.3) (xy 144.78 114.3))
+    (stroke (width 0) (type default))
+  )
+  (wire (pts (xy 132.08 92.71) (xy 120.65 92.71))
+    (stroke (width 0) (type default))
+  )
+  (wire (pts (xy 167.64 99.06) (xy 167.64 114.3))
+    (stroke (width 0) (type default))
+  )
+  (wire (pts (xy 160.02 99.06) (xy 160.02 114.3))
+    (stroke (width 0) (type default))
+  )
+  (wire (pts (xy 144.78 110.49) (xy 144.78 114.3))
+    (stroke (width 0) (type default))
+  )
+  (wire (pts (xy 144.78 83.82) (xy 144.78 87.63))
+    (stroke (width 0) (type default))
+  )
+  (wire (pts (xy 142.24 83.82) (xy 144.78 83.82))
+    (stroke (width 0) (type default))
+  )
+  (wire (pts (xy 120.65 92.71) (xy 120.65 114.3))
+    (stroke (width 0) (type default))
+  )
+  (wire (pts (xy 144.78 115.57) (xy 144.78 114.3))
+    (stroke (width 0) (type default))
+  )
+  (wire (pts (xy 124.46 100.33) (xy 124.46 83.82))
+    (stroke (width 0) (type default))
+  )
+  (wire (pts (xy 144.78 114.3) (xy 160.02 114.3))
+    (stroke (width 0) (type default))
+  )
+  (wire (pts (xy 132.08 100.33) (xy 124.46 100.33))
+    (stroke (width 0) (type default))
+  )
+  (wire (pts (xy 160.02 83.82) (xy 167.64 83.82))
+    (stroke (width 0) (type default))
+  )
+  (wire (pts (xy 142.24 87.63) (xy 142.24 83.82))
+    (stroke (width 0) (type default))
+  )
+  (wire (pts (xy 160.02 83.82) (xy 160.02 91.44))
+    (stroke (width 0) (type default))
+  )
+  (wire (pts (xy 120.65 114.3) (xy 142.24 114.3))
+    (stroke (width 0) (type default))
+  )
+  (wire (pts (xy 167.64 83.82) (xy 167.64 91.44))
+    (stroke (width 0) (type default))
+  )
+  (wire (pts (xy 144.78 80.01) (xy 144.78 83.82))
+    (stroke (width 0) (type default))
+  )
+  (wire (pts (xy 124.46 83.82) (xy 142.24 83.82))
+    (stroke (width 0) (type default))
+  )
+  (wire (pts (xy 142.24 110.49) (xy 142.24 114.3))
+    (stroke (width 0) (type default))
+  )
+  (wire (pts (xy 167.64 114.3) (xy 160.02 114.3))
+    (stroke (width 0) (type default))
+  )
+  (hierarchical_label "SCL" (shape input) (at 132.08 97.79 180) (fields_autoplaced)
+    (effects (font (size 1.27 1.27)) (justify right))
+  )
+  (hierarchical_label "SDA" (shape input) (at 132.08 95.25 180) (fields_autoplaced)
+    (effects (font (size 1.27 1.27)) (justify right))
+  )
+  (symbol (lib_id "power:GND") (at 144.78 115.57 0) (unit 1)
+    (in_bom yes) (on_board yes) (dnp no) (fields_autoplaced)
+    (property "Reference" "#PWR056" (at 144.78 121.92 0)
+      (effects (font (size 1.27 1.27)) hide)
+    )
+    (property "Value" "GND" (at 144.78 120.65 0)
+      (effects (font (size 1.27 1.27)))
+    )
+    (property "Footprint" "" (at 144.78 115.57 0)
+      (effects (font (size 1.27 1.27)) hide)
+    )
+    (property "Datasheet" "" (at 144.78 115.57 0)
+      (effects (font (size 1.27 1.27)) hide)
+    )
+    (pin "1")
+    (instances
+      (project "eesc"
+        (path "/ef2a3433-a5aa-4be9-bc22-47192e2652e7/495fd949-f99a-4be5-b307-d01e0baba967"
+          (reference "#PWR056") (unit 1)
+        )
+      )
+    )
+  )
+  (symbol (lib_id "Sensor_Motion:BMI160") (at 144.78 97.79 0) (unit 1)
+    (in_bom yes) (on_board yes) (dnp no) (fields_autoplaced)
+    (property "Reference" "U7" (at 146.7359 86.36 0)
+      (effects (font (size 1.27 1.27)) (justify left))
+    )
+    (property "Value" "BMI160" (at 146.7359 88.9 0)
+      (effects (font (size 1.27 1.27)) (justify left))
+    )
+    (property "Footprint" "Package_LGA:Bosch_LGA-14_3x2.5mm_P0.5mm" (at 144.78 97.79 0)
+      (effects (font (size 1.27 1.27)) hide)
+    )
+    (property "Datasheet" "https://www.bosch-sensortec.com/media/boschsensortec/downloads/datasheets/bst-bmi160-ds000.pdf" (at 127 76.2 0)
+      (effects (font (size 1.27 1.27)) hide)
+    )
+    (pin "1")
+    (pin "10")
+    (pin "11")
+    (pin "12")
+    (pin "13")
+    (pin "14")
+    (pin "2")
+    (pin "3")
+    (pin "4")
+    (pin "5")
+    (pin "6")
+    (pin "7")
+    (pin "8")
+    (pin "9")
+    (instances
+      (project "eesc"
+        (path "/ef2a3433-a5aa-4be9-bc22-47192e2652e7/495fd949-f99a-4be5-b307-d01e0baba967"
+          (reference "U7") (unit 1)
+        )
+      )
+    )
+  )
+  (symbol (lib_id "Device:C") (at 167.64 95.25 0) (unit 1)
+    (in_bom yes) (on_board yes) (dnp no)
+    (property "Reference" "C51" (at 168.91 92.71 0)
+      (effects (font (size 1.27 1.27)) (justify left))
+    )
+    (property "Value" "2.2u" (at 168.91 97.79 0)
+      (effects (font (size 1.27 1.27)) (justify left))
+    )
+    (property "Footprint" "" (at 168.6052 99.06 0)
+      (effects (font (size 1.27 1.27)) hide)
+    )
+    (property "Datasheet" "~" (at 167.64 95.25 0)
+      (effects (font (size 1.27 1.27)) hide)
+    )
+    (pin "1")
+    (pin "2")
+    (instances
+      (project "eesc"
+        (path "/ef2a3433-a5aa-4be9-bc22-47192e2652e7/495fd949-f99a-4be5-b307-d01e0baba967"
+          (reference "C51") (unit 1)
+        )
+      )
+    )
+  )
+  (symbol (lib_id "Device:C") (at 160.02 95.25 0) (unit 1)
+    (in_bom yes) (on_board yes) (dnp no)
+    (property "Reference" "C50" (at 161.29 92.71 0)
+      (effects (font (size 1.27 1.27)) (justify left))
+    )
+    (property "Value" "2.2u" (at 161.29 97.79 0)
+      (effects (font (size 1.27 1.27)) (justify left))
+    )
+    (property "Footprint" "" (at 160.9852 99.06 0)
+      (effects (font (size 1.27 1.27)) hide)
+    )
+    (property "Datasheet" "~" (at 160.02 95.25 0)
+      (effects (font (size 1.27 1.27)) hide)
+    )
+    (pin "1")
+    (pin "2")
+    (instances
+      (project "eesc"
+        (path "/ef2a3433-a5aa-4be9-bc22-47192e2652e7/495fd949-f99a-4be5-b307-d01e0baba967"
+          (reference "C50") (unit 1)
+        )
+      )
+    )
+  )
+  (symbol (lib_id "power:+3.3V") (at 144.78 80.01 0) (unit 1)
+    (in_bom yes) (on_board yes) (dnp no) (fields_autoplaced)
+    (property "Reference" "#PWR055" (at 144.78 83.82 0)
+      (effects (font (size 1.27 1.27)) hide)
+    )
+    (property "Value" "+3.3V" (at 144.78 76.2 0)
+      (effects (font (size 1.27 1.27)))
+    )
+    (property "Footprint" "" (at 144.78 80.01 0)
+      (effects (font (size 1.27 1.27)) hide)
+    )
+    (property "Datasheet" "" (at 144.78 80.01 0)
+      (effects (font (size 1.27 1.27)) hide)
+    )
+    (pin "1")
+    (instances
+      (project "eesc"
+        (path "/ef2a3433-a5aa-4be9-bc22-47192e2652e7/495fd949-f99a-4be5-b307-d01e0baba967"
+          (reference "#PWR055") (unit 1)
+        )
+      )
+    )
+  )
 )
