File: eesc/MCU.kicad_sch (KiCad schematic)
At the start: 0 parts

Commit message: Complete transistor stage
Parts:
- added C1, C10, C11, C2, C3, C4, C8, C9: 2.2u, symbol Device:C
- added C5: 100n, symbol Device:C
- added C6, C7: 15n, symbol Device:C
- added U1: STM32F405RGTx, Package_QFP:LQFP-64_10x10mm_P0.5mm, symbol MCU_ST_STM32F4:STM32F405RGTx
- added Y1: 8MHz, symbol Device:Crystal_GND23
Connections:
- new net: C4.1, U1.47 (VCAP_2)
- new net: C3.1, U1.31 (VCAP_1)
- new net +3.3V: C1.1, C10.1, C11.1, C2.1, C8.1, C9.1, U1.1 (VBAT), U1.13 (VDDA), U1.19 (VDD), U1.32 (VDD), U1.48 (VDD), U1.64 (VDD)
- new net GND: C1.2, C10.2, C11.2, C2.2, C3.2, C4.2, C5.2, C6.2, C7.2, C8.2, C9.2, U1.12 (VSSA), U1.18 (VSS), U1.60 (BOOT0), U1.63 (VSS), Y1.2, Y1.3
- new net NRST: C5.1, U1.7 (NRST)
- new net OSC_IN: C6.1, U1.5 (PH0), Y1.1
- new net OSC_OUT: C7.1, U1.6 (PH1), Y1.4
Other:
- note added: "Decoupling Capacitors Place near Vdd"
- note added: "Oscillator Circuit"
