File: eesc/Transistors.kicad_sch (KiCad schematic)
At the start: 0 parts

Commit message: Complete transistor stage
Parts:
- added C25, C34, C35, C36, C37, C38: 4.7u100v, symbol Device:C
- added J1: PH_A, symbol Connector_Generic:Conn_01x01
- added J2: PH_B, symbol Connector_Generic:Conn_01x01
- added J3: PH_C, symbol Connector_Generic:Conn_01x01
- added Q2, Q3, Q4, Q5, Q6, Q7: IRF7748L1, Package_DirectFET:DirectFET_L6, symbol Transistor_FET:IRF7748L1
- added R15, R16, R18, R19, R21, R22: 4.7, symbol Device:R
- added R17, R20, R23: 0.5m, symbol Device:R
Connections:
- new net: Q6.2 (G), R21.2
- new net: Q4.2 (G), R19.2
- new net: Q7.2 (G), R22.2
- new net: Q5.2 (G), R16.2
- new net: Q2.2 (G), R15.2
- new net: Q3.2 (G), R18.2
- new net GH_A: R15.1
- new net GH_B: R18.1
- new net GH_C: R21.1
- new net GL_A: R16.1
- new net GL_B: R19.1
- new net GL_C: R22.1
- new net GND: C25.2, C34.2, C35.2, C36.2, C37.2, C38.2, Q4.3 (S), Q5.3 (S), Q7.3 (S)
- new net IN_A+: Q2.3 (S), Q5.1 (D), R17.1
- new net IN_A-: J1.1 (Pin_1), R17.2
- new net IN_B+: Q3.3 (S), Q4.1 (D), R20.1
- new net IN_B-: J2.1 (Pin_1), R20.2
- new net IN_C+: Q6.3 (S), Q7.1 (D), R23.1
- new net IN_C-: J3.1 (Pin_1), R23.2
- new net V_SUPPLY: C25.1, C34.1, C35.1, C36.1, C37.1, C38.1, Q2.1 (D), Q3.1 (D), Q6.1 (D)
Other:
- note added: "Place 2 near per half-bridge"
