File: eesc/USB.kicad_sch (KiCad schematic)
At the start: 0 parts

Commit message: Most updated changes
Parts:
- added J4: USB_OTG, symbol Connector:USB_OTG
- added R31, R32: 22, symbol Device:R
Connections:
- new net: J4.2 (D-), R32.1
- new net: J4.3 (D+), R31.1
- new net +5V: J4.1 (VBUS)
- new net GND: J4.5 (GND), J4.6 (Shield)
- new net USB_D+: R31.2
- new net USB_D-: R32.2
- no-connect marks 0 -> 1
Changed lines of the file:
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@@
 (kicad_sch (version 20230121) (generator eeschema)
   (paper "A4")
+  (junction (at 115.57 83.82) (diameter 0) (color 0 0 0 0)
+  )
+  (no_connect (at 125.73 74.93))
+  (wire (pts (xy 115.57 80.01) (xy 115.57 83.82))
+    (stroke (width 0) (type default))
+  )
+  (wire (pts (xy 125.73 64.77) (xy 137.16 64.77))
+    (stroke (width 0) (type default))
+  )
+  (wire (pts (xy 137.16 69.85) (xy 140.97 69.85))
+    (stroke (width 0) (type default))
+  )
+  (wire (pts (xy 125.73 72.39) (xy 129.54 72.39))
+    (stroke (width 0) (type default))
+  )
+  (wire (pts (xy 118.11 83.82) (xy 118.11 80.01))
+    (stroke (width 0) (type default))
+  )
+  (wire (pts (xy 137.16 57.15) (xy 137.16 64.77))
+    (stroke (width 0) (type default))
+  )
+  (wire (pts (xy 125.73 69.85) (xy 129.54 69.85))
+    (stroke (width 0) (type default))
+  )
+  (wire (pts (xy 137.16 72.39) (xy 140.97 72.39))
+    (stroke (width 0) (type default))
+  )
+  (wire (pts (xy 115.57 83.82) (xy 118.11 83.82))
+    (stroke (width 0) (type default))
+  )
+  (hierarchical_label "USB_D+" (shape output) (at 140.97 69.85 0) (fields_autoplaced)
+    (effects (font (size 1.27 1.27)) (justify left))
+  )
+  (hierarchical_label "USB_D-" (shape output) (at 140.97 72.39 0) (fields_autoplaced)
+    (effects (font (size 1.27 1.27)) (justify left))
+  )
+  (symbol (lib_id "power:+5V") (at 137.16 57.15 0) (unit 1)
+    (in_bom yes) (on_board yes) (dnp no) (fields_autoplaced)
+    (property "Reference" "#PWR058" (at 137.16 60.96 0)
+      (effects (font (size 1.27 1.27)) hide)
+    )
+    (property "Value" "+5V" (at 137.16 53.34 0)
+      (effects (font (size 1.27 1.27)))
+    )
+    (property "Footprint" "" (at 137.16 57.15 0)
+      (effects (font (size 1.27 1.27)) hide)
+    )
+    (property "Datasheet" "" (at 137.16 57.15 0)
+      (effects (font (size 1.27 1.27)) hide)
+    )
+    (pin "1")
+    (instances
+      (project "eesc"
+        (path "/ef2a3433-a5aa-4be9-bc22-47192e2652e7/219c9e32-e282-428d-a4fa-0f43b167eba8"
+          (reference "#PWR058") (unit 1)
+        )
+      )
+    )
+  )
+  (symbol (lib_id "Device:R") (at 133.35 72.39 90) (unit 1)
+    (in_bom yes) (on_board yes) (dnp no)
+    (property "Reference" "R32" (at 132.08 74.93 90)
+      (effects (font (size 1.27 1.27)))
+    )
+    (property "Value" "22" (at 133.35 72.39 90)
+      (effects (font (size 1.27 1.27)))
+    )
+    (property "Footprint" "" (at 133.35 74.168 90)
+      (effects (font (size 1.27 1.27)) hide)
+    )
+    (property "Datasheet" "~" (at 133.35 72.39 0)
+      (effects (font (size 1.27 1.27)) hide)
+    )
+    (pin "1")
+    (pin "2")
+    (instances
+      (project "eesc"
+        (path "/ef2a3433-a5aa-4be9-bc22-47192e2652e7/219c9e32-e282-428d-a4fa-0f43b167eba8"
+          (reference "R32") (unit 1)
+        )
+      )
+    )
+  )
+  (symbol (lib_id "power:GND") (at 115.57 83.82 0) (unit 1)
+    (in_bom yes) (on_board yes) (dnp no) (fields_autoplaced)
+    (property "Reference" "#PWR057" (at 115.57 90.17 0)
+      (effects (font (size 1.27 1.27)) hide)
+    )
+    (property "Value" "GND" (at 115.57 88.9 0)
+      (effects (font (size 1.27 1.27)))
+    )
+    (property "Footprint" "" (at 115.57 83.82 0)
+      (effects (font (size 1.27 1.27)) hide)
+    )
+    (property "Datasheet" "" (at 115.57 83.82 0)
+      (effects (font (size 1.27 1.27)) hide)
+    )
+    (pin "1")
+    (instances
+      (project "eesc"
+        (path "/ef2a3433-a5aa-4be9-bc22-47192e2652e7/219c9e32-e282-428d-a4fa-0f43b167eba8"
+          (reference "#PWR057") (unit 1)
+        )
+      )
+    )
+  )
+  (symbol (lib_id "Device:R") (at 133.35 69.85 90) (unit 1)
+    (in_bom yes) (on_board yes) (dnp no)
+    (property "Reference" "R31" (at 132.08 67.31 90)
+      (effects (font (size 1.27 1.27)))
+    )
+    (property "Value" "22" (at 133.35 69.85 90)
+      (effects (font (size 1.27 1.27)))
+    )
+    (property "Footprint" "" (at 133.35 71.628 90)
+      (effects (font (size 1.27 1.27)) hide)
+    )
+    (property "Datasheet" "~" (at 133.35 69.85 0)
+      (effects (font (size 1.27 1.27)) hide)
+    )
+    (pin "1")
+    (pin "2")
+    (instances
+      (project "eesc"
+        (path "/ef2a3433-a5aa-4be9-bc22-47192e2652e7/219c9e32-e282-428d-a4fa-0f43b167eba8"
+          (reference "R31") (unit 1)
+        )
+      )
+    )
+  )
+  (symbol (lib_id "Connector:USB_OTG") (at 118.11 69.85 0) (unit 1)
+    (in_bom yes) (on_board yes) (dnp no) (fields_autoplaced)
+    (property "Reference" "J4" (at 118.11 58.42 0)
+      (effects (font (size 1.27 1.27)))
+    )
+    (property "Value" "USB_OTG" (at 118.11 60.96 0)
+      (effects (font (size 1.27 1.27)))
+    )
+    (property "Footprint" "" (at 121.92 71.12 0)
+      (effects (font (size 1.27 1.27)) hide)
+    )
+    (property "Datasheet" " ~" (at 121.92 71.12 0)
+      (effects (font (size 1.27 1.27)) hide)
+    )
+    (pin "1")
+    (pin "2")
+    (pin "3")
+    (pin "4")
+    (pin "5")
+    (pin "6")
+    (instances
+      (project "eesc"
+        (path "/ef2a3433-a5aa-4be9-bc22-47192e2652e7/219c9e32-e282-428d-a4fa-0f43b167eba8"
+          (reference "J4") (unit 1)
+        )
+      )
+    )
+  )
 )
