File: HighLevel/CAN.kicad_sch (KiCad schematic)
At the start: 4 parts, among them U1 TJA1051TK-3

Commit message: Final High Level + edits + footprint
Parts:
- C4: renamed from C1; footprint (none) -> Capacitor_SMD:C_0805_2012Metric
- C5: renamed from C2; footprint (none) -> Capacitor_SMD:C_0805_2012Metric
- R13: renamed from R1; footprint (none) -> Resistor_SMD:R_0805_2012Metric
- renumbered U1 to U2
Changed lines of the file:
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@@
   (symbol (lib_id "Device:C") (at 116.84 125.73 0) (unit 1)
     (in_bom yes) (on_board yes) (dnp no) (fields_autoplaced)
-    (property "Reference" "C1" (at 120.65 124.46 0)
+    (property "Reference" "C4" (at 120.65 124.46 0)
       (effects (font (size 1.27 1.27)) (justify left))
     )
@@
       (effects (font (size 1.27 1.27)) (justify left))
     )
-    (property "Footprint" "" (at 117.8052 129.54 0)
+    (property "Footprint" "Capacitor_SMD:C_0805_2012Metric" (at 117.8052 129.54 0)
       (effects (font (size 1.27 1.27)) hide)
     )
@@
       (project "HighLevel"
         (path "/26149e3f-2822-4531-a73b-0a61b71078cc/d37aac18-cba6-41cf-afef-0352e11a26d4"
-          (reference "C1") (unit 1)
+          (reference "C4") (unit 1)
         )
       )
@@
   (symbol (lib_id "Device:R") (at 160.02 111.76 0) (unit 1)
     (in_bom yes) (on_board yes) (dnp no) (fields_autoplaced)
-    (property "Reference" "R1" (at 162.56 110.49 0)
+    (property "Reference" "R13" (at 162.56 110.49 0)
       (effects (font (size 1.27 1.27)) (justify left))
     )
@@
       (effects (font (size 1.27 1.27)) (justify left))
     )
-    (property "Footprint" "" (at 158.242 111.76 90)
+    (property "Footprint" "Resistor_SMD:R_0805_2012Metric" (at 158.242 111.76 90)
       (effects (font (size 1.27 1.27)) hide)
     )
@@
       (project "HighLevel"
         (path "/26149e3f-2822-4531-a73b-0a61b71078cc/d37aac18-cba6-41cf-afef-0352e11a26d4"
-          (reference "R1") (unit 1)
+          (reference "R13") (unit 1)
         )
       )
@@
   (symbol (lib_id "Interface_CAN_LIN:TJA1051TK-3") (at 140.97 111.76 0) (unit 1)
     (in_bom yes) (on_board yes) (dnp no) (fields_autoplaced)
-    (property "Reference" "U1" (at 142.9259 99.06 0)
+    (property "Reference" "U2" (at 142.9259 99.06 0)
       (effects (font (size 1.27 1.27)) (justify left))
     )
@@
       (project "HighLevel"
         (path "/26149e3f-2822-4531-a73b-0a61b71078cc/d37aac18-cba6-41cf-afef-0352e11a26d4"
-          (reference "U1") (unit 1)
+          (reference "U2") (unit 1)
         )
       )
@@
   (symbol (lib_id "power:GND") (at 143.51 125.73 0) (unit 1)
     (in_bom yes) (on_board yes) (dnp no) (fields_autoplaced)
-    (property "Reference" "#PWR01" (at 143.51 132.08 0)
+    (property "Reference" "#PWR030" (at 143.51 132.08 0)
       (effects (font (size 1.27 1.27)) hide)
     )
@@
       (project "HighLevel"
         (path "/26149e3f-2822-4531-a73b-0a61b71078cc/d37aac18-cba6-41cf-afef-0352e11a26d4"
-          (reference "#PWR01") (unit 1)
+          (reference "#PWR030") (unit 1)
         )
       )
@@
   (symbol (lib_id "Device:C") (at 127 125.73 0) (unit 1)
     (in_bom yes) (on_board yes) (dnp no) (fields_autoplaced)
-    (property "Reference" "C2" (at 130.81 124.46 0)
+    (property "Reference" "C5" (at 130.81 124.46 0)
       (effects (font (size 1.27 1.27)) (justify left))
     )
@@
       (effects (font (size 1.27 1.27)) (justify left))
     )
-    (property "Footprint" "" (at 127.9652 129.54 0)
+    (property "Footprint" "Capacitor_SMD:C_0805_2012Metric" (at 127.9652 129.54 0)
       (effects (font (size 1.27 1.27)) hide)
     )
@@
       (project "HighLevel"
         (path "/26149e3f-2822-4531-a73b-0a61b71078cc/d37aac18-cba6-41cf-afef-0352e11a26d4"
-          (reference "C2") (unit 1)
+          (reference "C5") (unit 1)
         )
       )
@@
   (symbol (lib_id "power:+5V") (at 116.84 91.44 0) (unit 1)
     (in_bom yes) (on_board yes) (dnp no) (fields_autoplaced)
-    (property "Reference" "#PWR02" (at 116.84 95.25 0)
+    (property "Reference" "#PWR029" (at 116.84 95.25 0)
       (effects (font (size 1.27 1.27)) hide)
     )
@@
       (project "HighLevel"
         (path "/26149e3f-2822-4531-a73b-0a61b71078cc/d37aac18-cba6-41cf-afef-0352e11a26d4"
-          (reference "#PWR02") (unit 1)
+          (reference "#PWR029") (unit 1)
         )
       )

Commit message: Fix all errors
Changed lines of the file:
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@@
   (junction (at 139.7 125.73) (diameter 0) (color 0 0 0 0)
+  )
+  (junction (at 127 114.3) (diameter 0) (color 0 0 0 0)
   )
   (junction (at 143.51 125.73) (diameter 0) (color 0 0 0 0)
@@
         )
       )
+    )
+  )
+  (symbol (lib_id "power:PWR_FLAG") (at 127 114.3 0) (unit 1)
+    (in_bom yes) (on_board yes) (dnp no)
+    (property "Reference" "#FLG06" (at 127 112.395 0)
+      (effects (font (size 1.27 1.27)) hide)
+    )
+    (property "Value" "PWR_FLAG" (at 123.19 110.49 0)
+      (effects (font (size 1.27 1.27)))
+    )
+    (property "Footprint" "" (at 127 114.3 0)
+      (effects (font (size 1.27 1.27)) hide)
+    )
+    (property "Datasheet" "~" (at 127 114.3 0)
+      (effects (font (size 1.27 1.27)) hide)
+    )
+    (pin "1")
+    (instances
+      (project "HighLevel"
+        (path "/26149e3f-2822-4531-a73b-0a61b71078cc/d37aac18-cba6-41cf-afef-0352e11a26d4"
+          (reference "#FLG06") (unit 1)
+        )
+      )
