File: HighLevel/driver.kicad_sch (KiCad schematic)
At the start: 41 parts, among them J1 UCC27210DDA, J2 UCC27210DDA, J3 UCC27210DDA, U1 MCP16311MS, U2 MCP16311MS, U3 MC74VHC1GT66, U4 MC74VHC1GT66, U5 MC74VHC1GT66

Commit message: Final High Level + edits + footprint
Parts:
- renumbered C11 to C17, C10 to C18, C1 to C19, C7 to C20, C2 to C21, C12 to C22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
Connections:
- net SENS_2: no longer C32.1, R22.1, R23.1
- new net SENS_3: C32.1, R22.1, R23.1
