File: HighLevel/power_v2.kicad_sch (KiCad schematic)
At the start: 90 parts, among them J1 Conn_01x01, J2 Conn_01x01, J3 Conn_01x01, J4 Conn_01x01, J5 Conn_01x01, J6 Conn_01x01, Q1 IRF7759L2, Q10 IRF7759L2, Q11 IRF7759L2, Q12 IRF7759L2, Q13 IRF7759L2, Q14 IRF7759L2, Q15 IRF7759L2, Q16 IRF7759L2, Q17 IRF7759L2, Q18 IRF7759L2, Q2 IRF7759L2, Q3 IRF7759L2, Q4 IRF7759L2, Q5 IRF7759L2, Q6 IRF7759L2, Q7 IRF7759L2, Q8 IRF7759L2, Q9 IRF7759L2, U1 INA240A4PW, U17 MC74VHC1GT66, U18 MC74VHC1GT66, U19 MC74VHC1GT66, U2 INA240A4PW, U3 INA240A4PW

Commit message: Final High Level + edits + footprint
Parts:
- All_Capacitors, All_Capacitors1, All_Capacitors2, C1, C10, C11, C12, C13, C14, C15, C16, C2, C20, C21, C3, C4, C5, C6, C7, C8, C9: footprint (none) -> Capacitor_SMD:C_0805_2012Metric
- R1, R10, R11, R2, R4, R5, R6, R7, R9, r12, r3, r8: footprint (none) -> Resistor_SMD:R_0805_2012Metric

Commit message: Fix all errors
Parts:
- renumbered 0.0005 to 0.1, 0.1 to 0.2, 0.2 to 0.3, All_Capacitors to All_Capacitors1, All_Capacitors1 to All_Capacitors2, All_Capacitors2 to All_Capacitors3, C23 to C36, C1 to C37, C73 to C38, C17 to C39, C74 to C40, C75 to C41, C5 to C42, C2 to C43, C6 to C44, C3 to C45, C7 to C46, C26 to C47, C29 to C48, C4 to C49, C32 to C50, C33 to C51, C35 to C52, C18 to C53, C76 to C54, C36 to C55, C8 to C56, C9 to C57, C10 to C58, C11 to C59, C12 to C60, C13 to C61, C19 to C62, C77 to C63, C14 to C64, C15 to C65, C16 to C66, C20 to C67, C21 to C68, J1 to J11, J2 to J12, J3 to J13, J4 to J14, J5 to J15, J6 to J16, Q9 to Q10, Q10 to Q11, Q11 to Q12, Q12 to Q13, Q13 to Q14, Q14 to Q15, Q15 to Q16, Q16 to Q17, Q17 to Q18, Q18 to Q19, Q1 to Q2, Q4 to Q3, Q2 to Q4, Q3 to Q6, Q6 to Q7, Q7 to Q8, Q8 to Q9, R21 to R26, R22 to R27, R1 to R28, R2 to R29, R4 to R30, R49 to R31, R50 to R32, R17 to R34, R51 to R35, R52 to R36, R5 to R37, R6 to R38, R7 to R39, R18 to R41, R9 to R42, R10 to R43, R11 to R44, R19 to R46, U17 to U10, U2 to U11, U18 to U12, U3 to U13, U19 to U14, U1 to U9, r3 to r33, r8 to r40, r12 to r45
Connections:
- net C_A: now also U9.8
- net C_B: now also U11.8
- net C_C: now also U13.8
- net GND: no longer C37.1, U9.5 (V+), U9.6 (REF2)
- net VCC: now also C37.1, C49.1, C61.1, U11.5 (V+), U11.6 (REF2), U13.5 (V+), U13.6 (REF2), U9.5 (V+), U9.6 (REF2)

Commit message: Update power schematic to use TO-263 transistor
Parts:
- removed 0.1, 0.2, 0.3: 0.0005, symbol Device:R
- removed C42, C44, C45, C46, C56, C57, C58, C59, C60, C64, C65, C66, C67, C68: C, Capacitor_SMD:C_0805_2012Metric, symbol Device:C
- removed C47, C48: 470u_80V, Capacitor_THT:C_Radial_D16.0mm_H31.5mm_P7.50mm, symbol Device:C_Polarized_Small_US
- removed C49, C61: 2.2u, Capacitor_SMD:C_0805_2012Metric, symbol Device:C
- removed Q10, Q11, Q12, Q13, Q14, Q15, Q16, Q17, Q18, Q19, Q2, Q3, Q4, Q5, Q6, Q7, Q8, Q9: IRF7759L2, Package_DirectFET:DirectFET_L8, symbol Transistor_FET:IRF7759L2
- removed R37, R38, R42, R43: 0.0005, Resistor_SMD:R_0805_2012Metric, symbol Device:R
- removed R39, R44, r40, r45: 1R, Resistor_SMD:R_0805_2012Metric, symbol Device:R
- removed U13: INA240A4PW, Package_SO:TSSOP-8_4.4x3mm_P0.65mm, symbol Amplifier_Current:INA240A4PW
- added C37, C38: C, Capacitor_SMD:C_0805_2012Metric, symbol Device:C
- added C40, C41: 2.2u, Capacitor_SMD:C_0805_2012Metric, symbol Device:C
- added Q2, Q3, Q4, Q5, Q6, Q7: IPB039N10N3G, Package_TO_SOT_SMD:TO-263-6, symbol PCM_Transistor_MOSFET_AKL:IPB039N10N3G
- added R27, r33, r34: 1R, Resistor_SMD:R_0805_2012Metric, symbol Device:R
- added R30, R31: 0.005, Resistor_SMD:R_0805_2012Metric, symbol Device:R
- added U10: INA240A4PW, Package_SO:TSSOP-8_4.4x3mm_P0.65mm, symbol Amplifier_Current:INA240A4PW
- R28: value 0.0005 -> 1R
- R29: value 0.0005 -> 0.005
- U12: renamed from U10; footprint SOT95P275X110-5N -> Package_TO_SOT_SMD:SOT-353_SC-70-5
- U13: renamed from U12; footprint SOT95P275X110-5N -> Package_TO_SOT_SMD:SOT-353_SC-70-5
- U14: footprint SOT95P275X110-5N -> Package_TO_SOT_SMD:SOT-353_SC-70-5
- renumbered C43 to C36, C37 to C39, C41 to C42, C54 to C43, C63 to C44, C39 to C45, C53 to C46, C62 to C47, C50 to C48, C51 to C49, C52 to C50, C55 to C51, C36 to C52, C38 to C53, C40 to C54, R30 to R26, R34 to R35, R41 to R36, R46 to R37, R26 to R38, R31 to R39, R35 to R40, R27 to R41, R32 to R42, R36 to R43, r33 to r32
Connections:
- net C_B: now also U10.8; no longer U11.8
- net C_C: now also U11.8
- net GH_B: now also R27.2
- net GH_C: now also R28.2
- net GL_B: now also r33.1
- net GL_C: now also r34.1
- net GND: now also C37.2, C38.2, C40.2, C41.2, Q5.2 (S), Q5.3 (S), Q5.5 (S), Q5.6 (S), Q5.7 (S), Q6.2 (S), Q6.3 (S), Q6.5 (S), Q6.6 (S), Q6.7 (S), Q7.2 (S), Q7.3 (S), Q7.5 (S), Q7.6 (S), Q7.7 (S), U10.1 (GND), U10.4 (GND), U10.7 (REF1)
- net SH_A: now also R29.1, U9.2 (+), Q2.2 (S), Q2.3 (S), Q2.5 (S), Q2.6 (S), Q2.7 (S), Q5.4 (D); no longer r32.2
- net SH_B: now also Q3.2 (S), Q3.3 (S), Q3.5 (S), Q3.6 (S), Q3.7 (S), Q6.4 (D), R30.1, U10.2 (+)
- net SH_C: now also U11.2 (+), Q4.2 (S), Q4.3 (S), Q4.5 (S), Q4.6 (S), Q4.7 (S), Q7.4 (D), R31.1
- net VCC: now also C40.1, C41.1, U10.5 (V+), U10.6 (REF2)
- net V_IN: now also Q2.4 (D), Q3.4 (D), Q4.4 (D); no longer All_Capacitors1.1, All_Capacitors2.1, All_Capacitors3.1, C36.1, R26.1
- net at U11.3 (-): now also R31.2
- net at R29.2, U9.3 (-): no longer R28.2
- new net: All_Capacitors1.1, C36.1, Q2.1 (G), R26.1
- new net: All_Capacitors3.1, C38.1, Q4.1 (G), R28.1
- new net: Q5.1 (G), r32.2
- new net: R30.2, U10.3 (-)
- new net: Q7.1 (G), r34.2
- new net: All_Capacitors2.1, C37.1, Q3.1 (G), R27.1
- new net: Q6.1 (G), r33.2
Other:
- moved on the sheet: All_Capacitors1
